Commit message: Started Base of Robot In URDF

File: src/REPO_NAME_description/urdf/parts/swerve_axle.xacro (robot description, xacro)
@@ -36,4 +36,5 @@
                 <origin xyz="0 -${wheel_pos_y} 0" rpy="0 ${pi/4} ${pi/2}" />
                 <geometry>
+                     <mesh filename="package://REPO_NAME_description/meshes/SwerveAxle.stl"/>
                 </geometry>
                 <material name="yellow" />
