Commit message: Hopefully working URDF setup (meshes do not work)

File: src/repo_name_description/urdf/parts/swerve_axle.xacro (robot description, xacro)
@@ -36,5 +36,6 @@
                 <origin xyz="0 -${wheel_pos_y} 0" rpy="0 ${pi/4} ${pi/2}" />
                 <geometry>
-                     <mesh filename="package://REPO_NAME_description/meshes/SwerveAxle.stl"/>
+                    <!-- <cylinder length="${wheel_length}" radius="${wheel_radius}"/> -->
+                    <mesh filename="file:///../meshes/SwerveWheel.stl" />
                 </geometry>
                 <material name="yellow" />
@@ -43,5 +44,5 @@
                 <origin xyz="0 0 0" rpy="${pi / 2} 0 0"/>
                 <geometry>
-                    <cylinder  length="${wheel_length}" radius="${wheel_radius}"/>
+                    <cylinder length="${wheel_length}" radius="${wheel_radius}"/>
                 </geometry>
             </collision>

Commit message: Actually made the ROS workspace work for the packages ( they were missing the share directory ☺ )

File: src/repo_name_description/urdf/parts/swerve_axle.xacro (robot description, xacro)
@@ -37,5 +37,5 @@
                 <geometry>
                     <!-- <cylinder length="${wheel_length}" radius="${wheel_radius}"/> -->
-                    <mesh filename="file:///../meshes/SwerveWheel.stl" />
+                    <mesh filename="package://repo_name_description/meshes/SwerveWheel.stl"/>
                 </geometry>
                 <material name="yellow" />

File: src/repo_name_description/urdf/robot.urdf (robot description, URDF)
Before this commit: robot REPO_NAME, 3 links, 2 joints
Links:
- link front_left_wheel_link: geometry collision cylinder length=0.0381 radius=0.0508; visual mesh filename=package://repo_name_description/meshes/SwerveWheel.stl

File: src/repo_name_description/urdf/robot.urdf.xacro (robot description, xacro)
@@ -1,6 +1,6 @@
 <?xml version="1.0"?>
 <robot name="REPO_NAME" xmlns:xacro="http://www.ros.org/wiki/xacro">
-  <xacro:include filename="parts/swerve_axle.xacro" />
-  <xacro:include filename="util/macros.xacro" />
+  <xacro:include filename="$(find repo_name_description)/urdf/parts/swerve_axle.xacro" />
+  <xacro:include filename="$(find repo_name_description)/urdf/util/macros.xacro" />
   <link name="base_link"></link>
   <xacro:swerve_axle prefix="front_left" parent="base_link">

Commit message: Actually Made Wheel Upright

File: src/repo_name_description/urdf/parts/swerve_axle.xacro (robot description, xacro)
@@ -34,5 +34,5 @@
         <link name="${prefix}_wheel_link">
             <visual>
-                <origin xyz="0 -${wheel_pos_y} 0" rpy="0 ${pi/4} ${pi/2}" />
+                <origin xyz="0 -${wheel_pos_y} 0" rpy="0 0 ${pi/2}" />
                 <geometry>
                     <!-- <cylinder length="${wheel_length}" radius="${wheel_radius}"/> -->

Commit message: Tested Wheel Hitbox And Fixed Offset

File: src/repo_name_description/urdf/parts/swerve_axle.xacro (robot description, xacro)
@@ -8,9 +8,4 @@
     <xacro:property name="wheel_length" value="0.0381" />
     <xacro:property name="wheel_mass" value="0.23133211" />
-    <!-- Wheel Properties -->
-    <!-- NOTE: The below values are **guesses**-->
-    <!-- NOTE: Pretty good **guesses**-->
-    <xacro:property name="wheel_pos_y" value="0.022"/>
-    <xacro:property name="wheel_pos_z" value="0.063"/>
     <xacro:macro name="swerve_axle" params="prefix parent *origin">
         <link name="${prefix}_axle_link">
@@ -34,7 +29,6 @@
         <link name="${prefix}_wheel_link">
             <visual>
-                <origin xyz="0 -${wheel_pos_y} 0" rpy="0 0 ${pi/2}" />
+                <origin xyz="0 0 0" rpy="0 0 ${pi/2}" />
                 <geometry>
-                    <!-- <cylinder length="${wheel_length}" radius="${wheel_radius}"/> -->
                     <mesh filename="package://repo_name_description/meshes/SwerveWheel.stl"/>
                 </geometry>
@@ -54,5 +48,5 @@
             <parent link="${prefix}_axle_link" />
             <child link="${prefix}_wheel_link" />
-            <origin xyz="0 0 -${wheel_pos_z}" rpy="0 0 0"/>
+            <origin xyz="0 0 0" rpy="0 0 0"/>
             <axis xyz="0 1 0" />
             <dynamics friction="0.1" />

File: src/repo_name_description/urdf/robot.urdf (robot description, URDF)
Before this commit: robot REPO_NAME, 3 links, 2 joints
Joints:
- joint front_left_wheel_joint: origin xyz=0 0 -0.063 rpy=0 0 0 -> xyz=0 0 0 rpy=0 0 0

File: src/repo_name_description/urdf/robot.urdf.xacro (robot description, xacro)
@@ -3,4 +3,5 @@
   <xacro:include filename="$(find repo_name_description)/urdf/parts/swerve_axle.xacro" />
   <xacro:include filename="$(find repo_name_description)/urdf/util/macros.xacro" />
+  <xacro:include filename="$(find repo_name_description)/urdf/util/materials.xacro" />
   <link name="base_link"></link>
   <xacro:swerve_axle prefix="front_left" parent="base_link">

Commit message: Added Swerve Axle to Urdf

File: src/repo_name_description/urdf/parts/swerve_axle.xacro (robot description, xacro)
@@ -8,9 +8,11 @@
     <xacro:property name="wheel_length" value="0.0381" />
     <xacro:property name="wheel_mass" value="0.23133211" />
+    <xacro:property name="wheel_z_offset" value="-0.0425"/>
     <xacro:macro name="swerve_axle" params="prefix parent *origin">
         <link name="${prefix}_axle_link">
             <visual>
-                <origin xyz="0 0 0" rpy="${pi} 0 ${pi/2}" />
+                <origin xyz="0 0 0" rpy="0 0 0" />
                 <geometry>
+                    <mesh filename="package://repo_name_description/meshes/SwerveAxle.stl"/>
                 </geometry>
                 <material name="blue" />
@@ -48,5 +50,6 @@
             <parent link="${prefix}_axle_link" />
             <child link="${prefix}_wheel_link" />
-            <origin xyz="0 0 0" rpy="0 0 0"/>
+            <!-- <NOTE!!! This is a GUESS to offset the actual wheel onto the center of axle.> -->
+            <origin xyz="0 0 ${wheel_z_offset}" rpy="0 0 0"/>
             <axis xyz="0 1 0" />
             <dynamics friction="0.1" />
