Commit message: Added swerve chassis and positioned wheels.

File: src/repo_name_description/urdf/robot.urdf (robot description, URDF)
Before this commit: robot REPO_NAME, 3 links, 2 joints
Links:
- added link back_left_axle_link, mass 0.23739; visual mesh filename=package://repo_name_description/meshes/SwerveAxle.stl
- added link back_left_wheel_link, mass 0.23133211; collision cylinder length=0.0381 radius=0.0508; visual mesh filename=package://repo_name_description/meshes/SwerveWheel.stl
- added link back_right_axle_link, mass 0.23739; visual mesh filename=package://repo_name_description/meshes/SwerveAxle.stl
- added link back_right_wheel_link, mass 0.23133211; collision cylinder length=0.0381 radius=0.0508; visual mesh filename=package://repo_name_description/meshes/SwerveWheel.stl
- added link d_chassis_link, mass 19.0508795; collision box size=0.661 0.661 0.05588; visual mesh filename=package://repo_name_description/meshes/SwerveChassis.stl
- added link front_right_axle_link, mass 0.23739; visual mesh filename=package://repo_name_description/meshes/SwerveAxle.stl
- added link front_right_wheel_link, mass 0.23133211; collision cylinder length=0.0381 radius=0.0508; visual mesh filename=package://repo_name_description/meshes/SwerveWheel.stl
- link front_left_axle_link: geometry visual mesh filename=package://repo_name_description/meshes/SwerveAxle.stl
Joints:
- added joint back_left_axle_joint: type continuous, parent base_link, child back_left_axle_link, origin xyz= .25 .25 .05 rpy=0 0 0, axis 0 0 -1
- added joint back_left_wheel_joint: type continuous, parent back_left_axle_link, child back_left_wheel_link, origin xyz=0 0 -0.0425 rpy=0 0 0, axis 0 1 0
- added joint back_right_axle_joint: type continuous, parent base_link, child back_right_axle_link, origin xyz= -.25 -.25 .05 rpy=0 0 0, axis 0 0 -1
- added joint back_right_wheel_joint: type continuous, parent back_right_axle_link, child back_right_wheel_link, origin xyz=0 0 -0.0425 rpy=0 0 0, axis 0 1 0
- added joint d_chassis_joint: type fixed, parent base_link, child d_chassis_link, origin xyz=0 0 0 rpy=0 0 0
- added joint front_right_axle_joint: type continuous, parent base_link, child front_right_axle_link, origin xyz= .25 -.25 .05 rpy=0 0 0, axis 0 0 -1
- added joint front_right_wheel_joint: type continuous, parent front_right_axle_link, child front_right_wheel_link, origin xyz=0 0 -0.0425 rpy=0 0 0, axis 0 1 0
- joint front_left_axle_joint: origin xyz= 0 0 0 rpy=0 0 0 -> xyz= -.25 .25 .05 rpy=0 0 0
- joint front_left_wheel_joint: origin xyz=0 0 0 rpy=0 0 0 -> xyz=0 0 -0.0425 rpy=0 0 0

File: src/repo_name_description/urdf/robot.urdf.xacro (robot description, xacro)
@@ -1,10 +1,24 @@
 <?xml version="1.0"?>
 <robot name="REPO_NAME" xmlns:xacro="http://www.ros.org/wiki/xacro">
-  <xacro:include filename="$(find repo_name_description)/urdf/parts/swerve_axle.xacro" />
   <xacro:include filename="$(find repo_name_description)/urdf/util/macros.xacro" />
   <xacro:include filename="$(find repo_name_description)/urdf/util/materials.xacro" />
+  <xacro:include filename="$(find repo_name_description)/urdf/parts/swerve_chassis.xacro" />
+  <xacro:include filename="$(find repo_name_description)/urdf/parts/swerve_axle.xacro" />
+  <xacro:property name="axle_pos" value="2" />
   <link name="base_link"></link>
+  <xacro:square_chassis prefix="d" parent="base_link">
+    <origin xyz="0 0 0" rpy="0 0 0" />
+  </xacro:square_chassis>
   <xacro:swerve_axle prefix="front_left" parent="base_link">
-    <origin xyz=" 0 0 0" rpy="0 0 0" />
+    <origin xyz=" -.25 .25 .05" rpy="0 0 0" />
+  </xacro:swerve_axle>
+    <xacro:swerve_axle prefix="front_right" parent="base_link">
+    <origin xyz=" .25 -.25 .05" rpy="0 0 0" />
+  </xacro:swerve_axle>
+    <xacro:swerve_axle prefix="back_left" parent="base_link">
+    <origin xyz=" .25 .25 .05" rpy="0 0 0" />
+  </xacro:swerve_axle>
+    <xacro:swerve_axle prefix="back_right" parent="base_link">
+    <origin xyz=" -.25 -.25 .05" rpy="0 0 0" />
   </xacro:swerve_axle>
 </robot>
